File: KiCad/GR_PT2399_Breakout.kicad_pcb (KiCad board)
At the start: 2 copper layers, 49.2 x 65.2 mm, 48 parts, among them J1 Conn_01x02, J2 Conn_01x04, J3 Conn_01x02, J4 Conn_01x03, J5 Conn_01x02, Q1 2N3904, Q2 2N3904, U1 LM7805_TO220, U2 PT2399

Commit message: Add files via upload
Parts:
- added R18: 1K, Resistor_THT:R_Axial_DIN0207_L6.3mm_D2.5mm_P10.16mm_Horizontal, F.Cu at (126.3, 111.0)
- C20: value 1uF -> 4.7uF
- moved C20 2.09 mm to (121.4, 117.8), turned to 270 degrees
Connections:
- Q2 pad 2: Net-(C20-Pad1) -> Net-(Q2-Pad2)
Routing:
- net Net-(Q2-Pad2): track 0.00 -> 27.2 mm
- net Net-(C20-Pad1): track 49.9 -> 24.8 mm
