File: KiCad/GR_PT2399_Breakout.sch (KiCad schematic (older format))
At the start: 47 parts, among them J1 Conn_01x02, J2 Conn_01x04, J3 Conn_01x02, J4 Conn_01x03, J5 Conn_01x02, Q1 2N3904, Q2 2N3904, U1 LM7805_TO220, U2 PT2399

Commit message: Add files via upload
Parts:
- added R18: 1K, Resistor_THT:R_Axial_DIN0207_L6.3mm_D2.5mm_P10.16mm_Horizontal, symbol Device:R_Small_US
Connections:
- net at C20.1, R14.2: now also R18.1; no longer Q2.2 (B)
- new net: Q2.2 (B), R18.2
Other:
- moved on the sheet: C20
Changed lines of the file:
@@
 L Device:CP1_Small C20
 U 1 1 65EBFCEB
-P 2575 5000
-F 0 "C20" H 2725 5000 50  0000 C CNN
-F 1 "4.7uF" H 2750 4925 50  0000 C CNN
-F 2 "Capacitor_THT:CP_Radial_D5.0mm_P2.50mm" H 2575 5000 50  0001 C CNN
-F 3 "~" H 2575 5000 50  0001 C CNN
-	1    2575 5000
+P 2425 5000
+F 0 "C20" H 2575 5000 50  0000 C CNN
+F 1 "4.7uF" H 2600 4925 50  0000 C CNN
+F 2 "Capacitor_THT:CP_Radial_D5.0mm_P2.50mm" H 2425 5000 50  0001 C CNN
+F 3 "~" H 2425 5000 50  0001 C CNN
+	1    2425 5000
 	1    0    0    -1
 $EndComp
@@
 L power:GNDREF #PWR023
 U 1 1 65EBFCF5
-P 2575 5175
-F 0 "#PWR023" H 2575 4925 50  0001 C CNN
-F 1 "GNDREF" H 2825 4900 50  0001 C CNN
-F 2 "" H 2575 5175 50  0001 C CNN
-F 3 "" H 2575 5175 50  0001 C CNN
-	1    2575 5175
-	1    0    0    -1
-$EndComp
-Wire Wire Line
-	2575 5175 2575 5100
+P 2425 5175
+F 0 "#PWR023" H 2425 4925 50  0001 C CNN
+F 1 "GNDREF" H 2675 4900 50  0001 C CNN
+F 2 "" H 2425 5175 50  0001 C CNN
+F 3 "" H 2425 5175 50  0001 C CNN
+	1    2425 5175
+	1    0    0    -1
+$EndComp
+Wire Wire Line
+	2425 5175 2425 5100
 $Comp
 L Device:R_POT_US R14
@@
 	2125 4775 2125 4900
 Wire Wire Line
-	2275 4625 2575 4625
-Wire Wire Line
-	2575 4900 2575 4625
-Connection ~ 2575 4625
-Wire Wire Line
-	2575 4625 2750 4625
+	2275 4625 2425 4625
+Wire Wire Line
+	2425 4900 2425 4625
+Connection ~ 2425 4625
+Wire Wire Line
+	2425 4625 2500 4625
 $Comp
 L Device:C_Small C8
@@
 Text Notes 8225 3125 0    75   ~ 0
 Feedback
+$Comp
+L Device:R_Small_US R18
+U 1 1 65D61112
+P 2600 4625
+F 0 "R18" V 2525 4700 50  0000 R CNN
+F 1 "1K" V 2450 4700 50  0000 R CNN
+F 2 "Resistor_THT:R_Axial_DIN0207_L6.3mm_D2.5mm_P10.16mm_Horizontal" H 2600 4625 50  0001 C CNN
+F 3 "~" H 2600 4625 50  0001 C CNN
+	1    2600 4625
+	0    -1   -1   0
+$EndComp
+Wire Wire Line
+	2700 4625 2750 4625
 $EndSCHEMATC
